File: video/video.kicad_sch (KiCad schematic)
At the start: 5 parts, among them J4 DB9FEM, P1 BNC, P2 BNC, P3 BNC, P8 BNC

Commit message: Add 9.0 fs
Parts:
- P1, P2, P3, P8: footprint Discret:SUBCLICK -> footprints:subclick
